Commit message: fix step and limit
Signed-off-by: Steve Jeong <how2soft@gmail.com>

File: urdf/prototype.urdf (robot description, URDF)
Before this commit: robot visual, 14 links, 13 joints
Joints:
- joint ch0: limit lower=-0.785398 upper=1.57075 effort=1000.0 velocity=0.5 -> lower=-1.26 upper=1.26 effort=1000.0 velocity=0.5
- joint ch1: limit lower=-0.785398 upper=1.57075 effort=1000.0 velocity=0.5 -> lower=-1.26 upper=1.26 effort=1000.0 velocity=0.5
- joint ch2: limit lower=-0.785398 upper=1.57075 effort=1000.0 velocity=0.5 -> lower=-1.26 upper=1.26 effort=1000.0 velocity=0.5
- joint ch3: limit lower=0 upper=3.14 effort=1000.0 velocity=0.5 -> lower=-1.26 upper=1.26 effort=1000.0 velocity=0.5
- joint ch4: limit lower=0 upper=3.14 effort=1000.0 velocity=0.5 -> lower=-1.26 upper=1.26 effort=1000.0 velocity=0.5
